File: Deurnode nieuw.sch (KiCad schematic (older format))
At the start: 34 parts, among them J1 EXT1, J12 Screw_Terminal_01x03, J14 Screw_Terminal_01x02, J15 Screw_Terminal_01x02, J18 BarrelJack_DC5.5F, J19 Jumper Use external 12V, J2 EXT2, J22 Force output ON, J3 Conn_01x08, J4 Screw_Terminal_01x03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

Commit message: started on re-routing PCB increasing clearance from mains and using netclasses
Connections:
- wire segments 165 -> 167
Changed lines of the file:
@@
 F 3 "~" H 8600 1350 50  0001 C CNN
 	1    8600 1350
-	1    0    0    -1
+	1    0    0    1
 $EndComp
 Wire Wire Line
 	7900 850  8200 850
-Wire Wire Line
-	8200 850  8200 1350
-Wire Wire Line
-	8200 1350 8400 1350
-Wire Wire Line
-	7800 1450 8400 1450
 Wire Wire Line
 	7700 850  7700 750
@@
 Text Notes 5800 5390 0    49   ~ 0
 GND
-Text Notes 8700 1085 0    49   ~ 0
+Text Notes 8700 1300 0    49   ~ 0
 NC
-Text Notes 8700 1190 0    49   ~ 0
+Text Notes 8700 1500 0    49   ~ 0
 NO
-Text Notes 8700 1290 0    49   ~ 0
+Text Notes 8700 1400 0    49   ~ 0
 Common
 Text Notes 8705 4035 0    49   ~ 0
@@
 Wire Wire Line
 	8300 2000 8300 2200
+Wire Wire Line
+	8200 1450 8400 1450
+Wire Wire Line
+	8200 850  8200 1450
+Wire Wire Line
+	8400 1350 8100 1350
+Wire Wire Line
+	8100 1350 8100 1450
+Wire Wire Line
+	8100 1450 7800 1450
 $EndSCHEMATC
